File: Final Project V1/Final Project V1.kicad_sch (KiCad schematic)
At the start: 4 parts, among them U1 AP2112K-3.3, U2 ESP32-S3-WROOM-1

Commit message: Finish power rail
Parts:
- removed C1, C2: CL21B105KBFNNNG, CL21B105KBFNNNG:CAPC2012X140N, symbol CL21B105KBFNNNG:CL21B105KBFNNNG
- added C1, C2, C3, C4: 1uF (1206), Capacitor_SMD:C_1206_3216Metric_Pad1.33x1.80mm_HandSolder, symbol Device:C
- added D1, D2: 1N5817, Diode_THT:D_DO-41_SOD81_P10.16mm_Horizontal, symbol Diode:1N5817
- added J1: 39299043, CONN_5566-04x2_MOL, symbol 39299043:39299043
- added R1, R2: 1k, Resistor_SMD:R_1206_3216Metric_Pad1.30x1.75mm_HandSolder, symbol Device:R
- added U3: BQ21040DBVR, BQ21040DBVR:SOT95P280X145-6N, symbol BQ21040DBVR:BQ21040DBVR
Connections:
- net 3.3V: now also C1.1
- net 5V: now also C3.1, D1.2 (A), U3.6 (VIN)
- net GND: now also C1.2, C2.2, C3.2, C4.1, J1.2, R1.1, U3.5 (GND)
- net at U1.1 (VIN), U1.3 (EN): now also C2.1, D1.1 (K), D2.1 (K)
- new net: C4.2, D2.2 (A), J1.1, U3.2 (OUT)
- new net: R1.2, U3.4 (ISET)
- new net: R2.1, U3.3 (~{CHG})
- new net Connector for thermistor: U3.1 (TS)
- new net Microcontroller Charge Read: R2.2
Other:
- note added: "Power Circuit"
- moved on the sheet: U1

Commit message: Worked on PCB
Parts:
- added C10: 10uF (1206), Capacitor_SMD:C_1206_3216Metric_Pad1.33x1.80mm_HandSolder, symbol Device:C
- added C5: 100nF (1206), Capacitor_SMD:C_1206_3216Metric_Pad1.33x1.80mm_HandSolder, symbol Device:C
- added C6, C9: 1uF (1206), Capacitor_SMD:C_1206_3216Metric_Pad1.33x1.80mm_HandSolder, symbol Device:C
- added JP1: SolderJumper_3_Open, Jumper:SolderJumper-3_P2.0mm_Open_TrianglePad1.0x1.5mm, symbol Jumper:SolderJumper_3_Open
- added Q1, Q2: SS8050-G, Package_TO_SOT_SMD:SOT-23, symbol Device:Q_NPN_BEC
- added R10, R15: 100k, Resistor_SMD:R_1206_3216Metric_Pad1.30x1.75mm_HandSolder, symbol Device:R
- added R11, R12, R13, R14: 10k, Resistor_SMD:R_1206_3216Metric_Pad1.30x1.75mm_HandSolder, symbol Device:R
- added R3, R6: 1k, Resistor_SMD:R_1206_3216Metric_Pad1.30x1.75mm_HandSolder, symbol Device:R
- added SW1, SW2: SW_Push, Button_Switch_SMD:SW_SPST_B3S-1000, symbol Switch:SW_Push
- added USB-C1: UJC-HP-3-SMT-TR, UJC_HP_3_SMT_TR:CUI_UJC-HP-3-SMT-TR, symbol UJC-HP-3-SMT-TR:UJC-HP-3-SMT-TR
- J1: footprint CONN_5566-04x2_MOL -> footprints:CONN_5566-04x2_MOL
Connections:
- net 3.3V: now also C10.2, C5.2, JP1.3 (B), R10.2, R15.2, R3.2; no longer U2.3 (EN)
- net GND: now also C10.1, C5.1, C6.1, C9.2, JP1.1 (A), SW1.1, SW2.1, USB-C1.A12 (GND), USB-C1.B12 (GND__1), USB-C1.S1 (SHIELD), USB-C1.S2 (SHIELD__1), USB-C1.S3 (SHIELD__2), USB-C1.S4 (SHIELD__3)
- net at U2.15 (IO3): now also R6.2
- net at U2.16 (IO46): now also R3.1
- net at U2.27 (IO0): now also C6.2, R10.1, R13.2, SW2.2
- net 5V: no longer names the net of C3.1, D1.2 (A), U3.6 (VIN)
- net 5V: now also USB-C1.A9 (V-BUS), USB-C1.B9 (V-BUS__1)
- new net: Q1.1 (B), R12.2
- new net: JP1.2 (C), R6.1
- new net: Q1.3 (C), R14.1
- new net: Q2.1 (B), R11.2
- new net: Q2.3 (C), R13.1
- new net Chip_PU: C9.1, R14.2, R15.1, SW1.2, U2.3 (EN)
- new net DTR: Q2.2 (E), R12.1
- new net RTS: Q1.2 (E), R11.1
Other:
- note added: "May be fucked up"
- moved on the sheet: U2

Commit message: Finish V1 Board
Parts:
- added J2: Conn_01x05_Pin, Connector_PinSocket_2.54mm:PinSocket_1x05_P2.54mm_Vertical, symbol Connector:Conn_01x05_Pin
- added J3: Conn_01x03_Pin, Connector_PinSocket_2.54mm:PinSocket_1x03_P2.54mm_Vertical, symbol Connector:Conn_01x03_Pin
- added J4, J5: Conn_01x02_Pin, Connector_PinSocket_2.54mm:PinSocket_1x02_P2.54mm_Vertical, symbol Connector:Conn_01x02_Pin
- added J6: Conn_02x09_Counter_Clockwise, Connector_PinSocket_2.54mm:PinSocket_2x09_P2.54mm_Vertical, symbol Connector_Generic:Conn_02x09_Counter_Clockwise
- added R4: 1k, Resistor_SMD:R_0805_2012Metric_Pad1.20x1.40mm_HandSolder, symbol Device:R
- added R5, R7, R8, R9: 10k, Resistor_SMD:R_0805_2012Metric_Pad1.20x1.40mm_HandSolder, symbol Device:R
- added SW3: SW_Push, Button_Switch_SMD:SW_SPST_B3S-1000, symbol Switch:SW_Push
- added SW4, SW5: SW_Wuerth_450301014042, Button_Switch_THT:SW_Slide-03_Wuerth-WS-SLTV_10x2.5x6.4_P2.54mm, symbol Switch:SW_Wuerth_450301014042
- added U4, U5: 2SJ652-1E, TO-220F-3SG_15P87X10P16_ONS, symbol 2SJ652-1E:2SJ652-1E
- R1, R10, R11, R12, R13, R14, R15, R2, R3, R6: footprint Resistor_SMD:R_1206_3216Metric_Pad1.30x1.75mm_HandSolder -> Resistor_SMD:R_0805_2012Metric_Pad1.20x1.40mm_HandSolder
Connections:
- net 3.3V: now also J3.3 (Pin_3), J5.2 (Pin_2), SW3.2, U4.3 (S), U5.3 (S)
- net DTR: now also J2.4 (Pin_4)
- net GND: now also J2.1 (Pin_1), J3.1 (Pin_1), J4.1 (Pin_1), J6.1 (Pin_1), R5.1, R7.1
- net Microcontroller Charge Read: now also U2.7 (IO7)
- net RTS: now also J2.5 (Pin_5)
- net at C3.1, D1.2 (A), U3.6 (VIN): now also SW4.2 (C); no longer USB-C1.A9 (V-BUS), USB-C1.B9 (V-BUS__1)
- net at C4.2, D2.2 (A), U3.2 (OUT): now also SW5.1 (B); no longer J1.1
- net D1: now reaches U2.10 (IO17)
- net D1: now also J6.8 (Pin_8)
- net D0: now reaches U2.11 (IO18)
- net D0: now also J6.11 (Pin_11)
- net VS: now reaches U2.17 (IO9)
- net VS: now also J6.3 (Pin_3)
- net HS: now reaches U2.18 (IO10)
- net HS: now also J6.16 (Pin_16)
- net PCLK: now reaches U2.19 (IO11)
- net PCLK: now also J6.4 (Pin_4)
- net MCLK: now reaches U2.20 (IO12)
- net MCLK: now also J6.15 (Pin_15)
- net D7: now reaches U2.21 (IO13)
- net D7: now also J6.5 (Pin_5)
- net D6: now reaches U2.22 (IO14)
- net D6: now also J6.14 (Pin_14)
- net D5: now reaches U2.23 (IO21)
- net D5: now also J6.6 (Pin_6)
- net D4: now reaches U2.24 (IO47)
- net D4: now also J6.13 (Pin_13)
- net Camera Power Signal: now reaches U2.25 (IO48)
- net Camera Power Signal: now also U4.1 (G)
- net Motor Power Signal: now reaches U2.26 (IO45)
- net Motor Power Signal: now also U5.1 (G)
- net Hall Read: now reaches U2.32 (IO39)
- net Hall Read: now also J3.2 (Pin_2)
- net Manual Feed: now reaches U2.33 (IO40)
- net Manual Feed: now also R4.1
- net RX: now reaches U2.36 (RXD0)
- net RX: now also J2.2 (Pin_2)
- net TX: now reaches U2.37 (TXD0)
- net TX: now also J2.3 (Pin_3)
- net SDA: now reaches U2.38 (IO2)
- net SDA: now also J6.17 (Pin_17), R8.2
- net SCL: now reaches U2.39 (IO1)
- net SCL: now also J6.2 (Pin_2), R9.2
- net D3: now reaches U2.8 (IO15)
- net D3: now also J6.7 (Pin_7)
- net D2: now reaches U2.9 (IO16)
- net D2: now also J6.12 (Pin_12)
- new net: J1.1, SW5.2 (C)
- new net: J5.1 (Pin_1), R5.2
- new net: R4.2, SW3.1
- new net: J6.10 (Pin_10), R7.2
- new net: SW4.1 (B), USB-C1.A9 (V-BUS), USB-C1.B9 (V-BUS__1)
- new net Camera Power: J6.18 (Pin_18), J6.9 (Pin_9), R8.1, R9.1, U4.2 (D)
- new net Motor Out: J4.2 (Pin_2), U5.2 (D)
Other:
- note added: "LED"

Commit message: Change socket headers to pins and use through-hole buttons. Need to try switch on pcb when arrives and change camera connector
Parts:
- removed J2: Conn_01x05_Pin, Connector_PinSocket_2.54mm:PinSocket_1x05_P2.54mm_Vertical, symbol Connector:Conn_01x05_Pin
- removed J3: Conn_01x03_Pin, Connector_PinSocket_2.54mm:PinSocket_1x03_P2.54mm_Vertical, symbol Connector:Conn_01x03_Pin
- removed J4, J5: Conn_01x02_Pin, Connector_PinSocket_2.54mm:PinSocket_1x02_P2.54mm_Vertical, symbol Connector:Conn_01x02_Pin
- removed SW1, SW2, SW3: SW_Push, Button_Switch_SMD:SW_SPST_B3S-1000, symbol Switch:SW_Push
- added J2: Conn_02x03_Counter_Clockwise, Connector_PinHeader_2.54mm:PinHeader_2x03_P2.54mm_Vertical, symbol Connector_Generic:Conn_02x03_Counter_Clockwise
- added J3: Conn_02x02_Counter_Clockwise, Connector_PinHeader_2.54mm:PinHeader_2x02_P2.54mm_Vertical, symbol Connector_Generic:Conn_02x02_Counter_Clockwise
- added J4, J5, J7: Conn_02x01, Connector_PinHeader_2.54mm:PinHeader_2x01_P2.54mm_Vertical, symbol Connector_Generic:Conn_02x01
- added R16: 10k, Resistor_SMD:R_0805_2012Metric_Pad1.20x1.40mm_HandSolder, symbol Device:R
- added SW3, SW6: 1825910-6, 1825910_6:SW_1825910-6-4, symbol 1825910-6:1825910-6
- C10: value 10uF (1206) -> 10uF (0805); footprint Capacitor_SMD:C_1206_3216Metric_Pad1.33x1.80mm_HandSolder -> Capacitor_SMD:C_0805_2012Metric_Pad1.18x1.45mm_HandSolder
- C5: value 100nF (1206) -> .1uF (0805); footprint Capacitor_SMD:C_1206_3216Metric_Pad1.33x1.80mm_HandSolder -> Capacitor_SMD:C_0805_2012Metric_Pad1.18x1.45mm_HandSolder
- R5: value 10k -> 1k
Connections:
- net 3.3V: now also J3.3 (Pin_3), J5.2 (Pin_2), J7.2 (Pin_2)
- net Chip_PU: now also SW3.3, SW3.4
- net DTR: now also J2.4 (Pin_4)
- net GND: now also J2.1 (Pin_1), J2.6 (Pin_6), J3.1 (Pin_1), J3.4 (Pin_4), J4.1 (Pin_1), R16.2, SW3.1, SW3.2, SW6.3, SW6.4
- net Hall Read: now also U2.5 (IO5), J3.2 (Pin_2); no longer U2.32 (IO39)
- net Manual Feed: now also R16.1
- net Motor Out: now also J4.2 (Pin_2)
- net RTS: now also J2.5 (Pin_5)
- net RX: now also J2.2 (Pin_2)
- net TX: now also J2.3 (Pin_3)
- net at C6.2, R10.1, R13.2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: now also SW6.1, SW6.2
- net at R5.2: now also J5.1 (Pin_1)
- net at R4.2: now also J7.1 (Pin_1)
Other:
- note added: "Dont solder"
- note removed: "May be fucked up"
- moved on the sheet: R5
